Commit message: pick & place

File: src/ur5_description/urdf/ur5_gripper_camera.xacro (robot description, xacro)
@@ -18,5 +18,5 @@
   <!-- Define RGB-D sensor -->
   <xacro:kinetic_rgb name="rgbd_camera" parent="base">
-    <origin xyz="0.1 0.0 1.2" rpy="${0.0 * deg_to_rad} ${70.0 * deg_to_rad} ${0.0 * deg_to_rad}"/>
+    <origin xyz="0.1 0.0 1.2" rpy="${0.0 * deg_to_rad} ${70.0 * deg_to_rad} ${90 * deg_to_rad}"/>
     <origin xyz="0 0 0" rpy="${-90 * deg_to_rad} ${0 * deg_to_rad} ${-90 * deg_to_rad}" />
   </xacro:kinetic_rgb>
